Commit message: sensor updates

File: body.urdf (robot description, URDF)
Before this commit: robot robot, 3 links, 2 joints
Links:
- removed link Link0
- removed link Link1
- removed link Link2
- added link BackLeg, mass 1; collision box size=1 1 1; visual box size=1 1 1
- added link FrontLeg, mass 1; collision box size=1 1 1; visual box size=1 1 1
- added link Torso, mass 1; collision box size=1 1 1; visual box size=1 1 1
Joints:
- removed joint Link0_Link1
- removed joint Link1_Link2
- added joint Torso_BackLeg: type revolute, parent Torso, child BackLeg, origin xyz=0.5 0 1 rpy=0 0 0, axis 0 1 0, limit lower=-3.14159 upper=3.14159 effort=0.0 velocity=0.0
- added joint Torso_FrontLeg: type revolute, parent Torso, child FrontLeg, origin xyz=1.5 0 1 rpy=0 0 0, axis 0 1 0, limit lower=-3.14159 upper=3.14159 effort=0.0 velocity=0.0

Commit message: quadruped updates

File: body.urdf (robot description, URDF)
Before this commit: robot robot, 3 links, 2 joints
Links:
- added link BackLower, mass 1; collision box size=0.2 0.2 1; visual box size=0.2 0.2 1
- added link FrontLower, mass 1; collision box size=0.2 0.2 1; visual box size=0.2 0.2 1
- added link LeftLeg, mass 1; collision box size=1 0.2 0.2; visual box size=1 0.2 0.2
- added link LeftLower, mass 1; collision box size=0.2 0.2 1; visual box size=0.2 0.2 1
- added link RightLeg, mass 1; collision box size=1 0.2 0.2; visual box size=1 0.2 0.2
- added link RightLower, mass 1; collision box size=0.2 0.2 1; visual box size=0.2 0.2 1
- link BackLeg: geometry collision box size=0.2 1 0.2; visual box size=0.2 1 0.2
- link FrontLeg: geometry collision box size=0.2 1 0.2; visual box size=0.2 1 0.2
Joints:
- added joint BackLeg_BackLower: type revolute, parent BackLeg, child BackLower, origin xyz=0 -1 0 rpy=0 0 0, axis 1 0 0, limit lower=-3.14159 upper=3.14159 effort=0.0 velocity=0.0
- added joint FrontLeg_FrontLower: type revolute, parent FrontLeg, child FrontLower, origin xyz=0 1 0 rpy=0 0 0, axis 1 0 0, limit lower=-3.14159 upper=3.14159 effort=0.0 velocity=0.0
- added joint LeftLeg_LeftLower: type revolute, parent LeftLeg, child LeftLower, origin xyz=1 0 0 rpy=0 0 0, axis 0 1 0, limit lower=-3.14159 upper=3.14159 effort=0.0 velocity=0.0
- added joint RightLeg_RightLower: type revolute, parent RightLeg, child RightLower, origin xyz=-1 0 0 rpy=0 0 0, axis 0 1 0, limit lower=-3.14159 upper=3.14159 effort=0.0 velocity=0.0
- added joint Torso_LeftLeg: type revolute, parent Torso, child LeftLeg, origin xyz=0.5 0 1 rpy=0 0 0, axis 0 1 0, limit lower=-3.14159 upper=3.14159 effort=0.0 velocity=0.0
- added joint Torso_RightLeg: type revolute, parent Torso, child RightLeg, origin xyz=-0.5 0 1 rpy=0 0 0, axis 0 1 0, limit lower=-3.14159 upper=3.14159 effort=0.0 velocity=0.0
- joint Torso_BackLeg: axis 0 1 0 -> 1 0 0; origin xyz=0.5 0 1 rpy=0 0 0 -> xyz=0 -0.5 1 rpy=0 0 0
- joint Torso_FrontLeg: axis 0 1 0 -> 1 0 0; origin xyz=1.5 0 1 rpy=0 0 0 -> xyz=0 0.5 1 rpy=0 0 0

Commit message: assignment 5 updates

File: body.urdf (robot description, URDF)
Before this commit: robot robot, 9 links, 8 joints
Links:
- removed link BackLeg
- removed link BackLower
- removed link FrontLeg
- removed link FrontLower
- removed link LeftLeg
- removed link LeftLower
- removed link RightLeg
- removed link RightLower
- added link BackLeft, mass 1; collision box size=0.2 0.2 1; visual box size=0.2 0.2 1
- added link BackRight, mass 1; collision box size=0.2 0.2 1; visual box size=0.2 0.2 1
- added link FrontLeft, mass 1; collision box size=0.2 0.2 1; visual box size=0.2 0.2 1
- added link FrontRight, mass 1; collision box size=0.2 0.2 1; visual box size=0.2 0.2 1
- link Torso: geometry collision box size=2 0.2 0.2; visual box size=2 0.2 0.2
Joints:
- removed joint BackLeg_BackLower
- removed joint FrontLeg_FrontLower
- removed joint LeftLeg_LeftLower
- removed joint RightLeg_RightLower
- removed joint Torso_BackLeg
- removed joint Torso_FrontLeg
- removed joint Torso_LeftLeg
- removed joint Torso_RightLeg
- added joint Torso_BackLeft: type revolute, parent Torso, child BackLeft, origin xyz=0.5 -0.1 1 rpy=0 0 0, axis 0 1 0, limit lower=-3.14159 upper=3.14159 effort=0.0 velocity=0.0
- added joint Torso_BackRight: type revolute, parent Torso, child BackRight, origin xyz=0.5 0.1 1 rpy=0 0 0, axis 0 1 0, limit lower=-3.14159 upper=3.14159 effort=0.0 velocity=0.0
- added joint Torso_FrontLeft: type revolute, parent Torso, child FrontLeft, origin xyz=-0.5 -0.1 1 rpy=0 0 0, axis 0 1 0, limit lower=-3.14159 upper=3.14159 effort=0.0 velocity=0.0
- added joint Torso_FrontRight: type revolute, parent Torso, child FrontRight, origin xyz=-0.5 0.1 1 rpy=0 0 0, axis 0 1 0, limit lower=-3.14159 upper=3.14159 effort=0.0 velocity=0.0

Commit message: HW 6 Snake Updates

File: body.urdf (robot description, URDF)
Before this commit: robot robot, 5 links, 4 joints
Links:
- removed link BackLeft
- removed link BackRight
- removed link FrontLeft
- removed link FrontRight
- removed link Torso
- added link 0, mass 1; collision box size=0.7559495928031804 0.9270842750800503 0.7584246941563578; visual box size=0.7559495928031804 0.9270842750800503 0.7584246941563578
- added link 1, mass 1; collision box size=0.9288868613081271 0.5965215132642716 0.9571439498515286; visual box size=0.9288868613081271 0.5965215132642716 0.9571439498515286
- added link 2, mass 1; collision box size=0.610623015956189 0.7096415027286564 0.9718549480210775; visual box size=0.610623015956189 0.7096415027286564 0.9718549480210775
- added link 3, mass 1; collision box size=0.8029157519237151 0.5843512728708717 0.8007368635530503; visual box size=0.8029157519237151 0.5843512728708717 0.8007368635530503
- added link 4, mass 1; collision box size=0.9524109415297304 0.7979097892485043 0.8862768061628525; visual box size=0.9524109415297304 0.7979097892485043 0.8862768061628525
- added link 5, mass 1; collision box size=0.5831901535206003 0.9733636849793972 0.8280015135880113; visual box size=0.5831901535206003 0.9733636849793972 0.8280015135880113
- added link 6, mass 1; collision box size=0.5947572993236623 0.9385768383960074 0.788902467302335; visual box size=0.5947572993236623 0.9385768383960074 0.788902467302335
- added link 7, mass 1; collision box size=0.7150983987175785 0.5331653036056712 0.6483228656137543; visual box size=0.7150983987175785 0.5331653036056712 0.6483228656137543
- added link 8, mass 1; collision box size=0.9664909291893141 0.516215338926408 0.5126349628362762; visual box size=0.9664909291893141 0.516215338926408 0.5126349628362762
Joints:
- removed joint Torso_BackLeft
- removed joint Torso_BackRight
- removed joint Torso_FrontLeft
- removed joint Torso_FrontRight
- added joint 0_1: type revolute, parent 0, child 1, origin xyz=-3.62202520359841 0 0.3792123470781789 rpy=0 0 0, axis 0 1 1, limit lower=-3.14159 upper=3.14159 effort=0.0 velocity=0.0
- added joint 1_2: type revolute, parent 1, child 2, origin xyz=0.9288868613081271 0 0 rpy=0 0 0, axis 0 1 1, limit lower=-3.14159 upper=3.14159 effort=0.0 velocity=0.0
- added joint 2_3: type revolute, parent 2, child 3, origin xyz=0.610623015956189 0 0 rpy=0 0 0, axis 0 1 1, limit lower=-3.14159 upper=3.14159 effort=0.0 velocity=0.0
- added joint 3_4: type revolute, parent 3, child 4, origin xyz=0.8029157519237151 0 0 rpy=0 0 0, axis 0 1 1, limit lower=-3.14159 upper=3.14159 effort=0.0 velocity=0.0
- added joint 4_5: type revolute, parent 4, child 5, origin xyz=0.9524109415297304 0 0 rpy=0 0 0, axis 0 1 1, limit lower=-3.14159 upper=3.14159 effort=0.0 velocity=0.0
- added joint 5_6: type revolute, parent 5, child 6, origin xyz=0.5831901535206003 0 0 rpy=0 0 0, axis 0 1 1, limit lower=-3.14159 upper=3.14159 effort=0.0 velocity=0.0
- added joint 6_7: type revolute, parent 6, child 7, origin xyz=0.5947572993236623 0 0 rpy=0 0 0, axis 0 1 1, limit lower=-3.14159 upper=3.14159 effort=0.0 velocity=0.0
- added joint 7_8: type revolute, parent 7, child 8, origin xyz=0.7150983987175785 0 0 rpy=0 0 0, axis 0 1 1, limit lower=-3.14159 upper=3.14159 effort=0.0 velocity=0.0

Commit message: HW 6 Snakes Last Updates

File: body.urdf (robot description, URDF)
Before this commit: robot robot, 9 links, 8 joints
Links:
- link 0: geometry collision box size=0.5282407194186273 0.7360883914904093 0.8663472596992636; visual box size=0.5282407194186273 0.7360883914904093 0.8663472596992636
- link 1: geometry collision box size=0.5741188043398946 0.8735452910295991 0.6273093833278324; visual box size=0.5741188043398946 0.8735452910295991 0.6273093833278324
- link 2: geometry collision box size=0.7843085973105834 0.74354718580087 0.5527219001297505; visual box size=0.7843085973105834 0.74354718580087 0.5527219001297505
- link 3: geometry collision box size=0.946698637989492 0.6822645106790555 0.8735443071400701; visual box size=0.946698637989492 0.6822645106790555 0.8735443071400701
- link 4: geometry collision box size=0.8296831624138096 0.5777602200935343 0.9544349994404857; visual box size=0.8296831624138096 0.5777602200935343 0.9544349994404857
- link 5: geometry collision box size=0.9817947522954504 0.5061441817515748 0.5957419079518766; visual box size=0.9817947522954504 0.5061441817515748 0.5957419079518766
- link 6: geometry collision box size=0.7431011464385565 0.8343465064675868 0.5856778018751386; visual box size=0.7431011464385565 0.8343465064675868 0.5856778018751386
- link 7: geometry collision box size=0.7955378435464546 0.5005661809959465 0.9567753926564982; visual box size=0.7955378435464546 0.5005661809959465 0.9567753926564982
- link 8: geometry collision box size=0.865334572771089 0.6053489360708226 0.7023306235610842; visual box size=0.865334572771089 0.6053489360708226 0.7023306235610842
Joints:
- joint 0_1: origin xyz=-3.62202520359841 0 0.3792123470781789 rpy=0 0 0 -> xyz=-3.7358796402906864 0 0.4331736298496318 rpy=0 0 0
- joint 1_2: origin xyz=0.9288868613081271 0 0 rpy=0 0 0 -> xyz=0.5741188043398946 0 0 rpy=0 0 0
- joint 2_3: origin xyz=0.610623015956189 0 0 rpy=0 0 0 -> xyz=0.7843085973105834 0 0 rpy=0 0 0
- joint 3_4: origin xyz=0.8029157519237151 0 0 rpy=0 0 0 -> xyz=0.946698637989492 0 0 rpy=0 0 0
- joint 4_5: origin xyz=0.9524109415297304 0 0 rpy=0 0 0 -> xyz=0.8296831624138096 0 0 rpy=0 0 0
- joint 5_6: origin xyz=0.5831901535206003 0 0 rpy=0 0 0 -> xyz=0.9817947522954504 0 0 rpy=0 0 0
- joint 6_7: origin xyz=0.5947572993236623 0 0 rpy=0 0 0 -> xyz=0.7431011464385565 0 0 rpy=0 0 0
- joint 7_8: origin xyz=0.7150983987175785 0 0 rpy=0 0 0 -> xyz=0.7955378435464546 0 0 rpy=0 0 0

Commit message: HW 7 updates

File: body.urdf (robot description, URDF)
Before this commit: robot robot, 9 links, 8 joints
Links:
- removed link 5
- removed link 6
- removed link 7
- removed link 8
- link 0: geometry collision box size=0.7965236154252942 0.5375184620693675 0.5417770483242674; visual box size=0.7965236154252942 0.5375184620693675 0.5417770483242674
- link 1: geometry collision box size=0.838574464283431 0.4688011037771848 0.35440994175372714; visual box size=0.838574464283431 0.4688011037771848 0.35440994175372714
- link 2: geometry collision box size=0.6990803240596797 0.22131939627457214 0.45525600415502515; visual box size=0.6990803240596797 0.22131939627457214 0.45525600415502515
- link 3: geometry collision box size=0.3790491448979757 0.7259155565165026 0.403311961282181; visual box size=0.3790491448979757 0.7259155565165026 0.403311961282181
- link 4: geometry collision box size=0.8117814183086364 0.11763949105382365 0.15247419560944386; visual box size=0.8117814183086364 0.11763949105382365 0.15247419560944386
Joints:
- removed joint 1_2
- removed joint 2_3
- removed joint 3_4
- removed joint 4_5
- removed joint 5_6
- removed joint 6_7
- removed joint 7_8
- added joint 0_2: type revolute, parent 0, child 2, origin xyz=0.3982618077126471 0.15231880376331192 0.14786657441217718 rpy=0 0 0, axis 0 1 1, limit lower=-3.14159 upper=3.14159 effort=0.0 velocity=0.0
- added joint 0_3: type revolute, parent 0, child 3, origin xyz=-0.18282078084885608 -0.26875923103468374 0.16149691452310025 rpy=0 0 0, axis 1 0 1, limit lower=-3.14159 upper=3.14159 effort=0.0 velocity=0.0
- added joint 0_4: type revolute, parent 0, child 4, origin xyz=0.3982618077126471 0.11335291441687195 0.02029945613171293 rpy=0 0 0, axis 0 1 1, limit lower=-3.14159 upper=3.14159 effort=0.0 velocity=0.0
- joint 0_1: origin xyz=-3.7358796402906864 0 0.4331736298496318 rpy=0 0 0 -> xyz=-0.3982618077126471 0.03604650011230143 0.08939324456205684 rpy=0 0 0

Commit message: HW8 First Try

File: body.urdf (robot description, URDF)
Before this commit: robot robot, 5 links, 4 joints
Links:
- link 0: geometry collision box size=1.1210310934486443 0.5454416751907422 0.9849061299035676; visual box size=1.1210310934486443 0.5454416751907422 0.9849061299035676
- link 1: geometry collision box size=0.2557703742904795 0.48564846894274594 1.124006305440842; visual box size=0.2557703742904795 0.48564846894274594 1.124006305440842
- link 2: geometry collision box size=1.409280422223762 0.021811760582099715 0.05779118820241419; visual box size=1.409280422223762 0.021811760582099715 0.05779118820241419
- link 3: geometry collision box size=1.0865641135754425 0.4116040987983699 0.06912677270542028; visual box size=1.0865641135754425 0.4116040987983699 0.06912677270542028
- link 4: geometry collision box size=0.13711092743813785 1.1102075107958906 0.38322189650920824; visual box size=0.13711092743813785 1.1102075107958906 0.38322189650920824
Joints:
- joint 0_1: axis 0 1 1 -> 1 1 0; origin xyz=-0.3982618077126471 0.03604650011230143 0.08939324456205684 rpy=0 0 0 -> xyz=0.04001758024304358 0.09857170190427922 0.9849061299035676 rpy=0 0 0
- joint 0_2: origin xyz=0.3982618077126471 0.15231880376331192 0.14786657441217718 rpy=0 0 0 -> xyz=-0.5605155467243221 -0.1903089767000891 0.6806745243426983 rpy=0 0 0
- joint 0_3: axis 1 0 1 -> 0 1 1; origin xyz=-0.18282078084885608 -0.26875923103468374 0.16149691452310025 rpy=0 0 0 -> xyz=0.5605155467243221 -0.15534274269175377 0.9060233358558663 rpy=0 0 0
- joint 0_4: axis 0 1 1 -> 1 0 1; origin xyz=0.3982618077126471 0.11335291441687195 0.02029945613171293 rpy=0 0 0 -> xyz=-0.39665305309138976 0.2727208375953711 0.17725037835031493 rpy=0 0 0

Commit message: HW8 Final Updates

File: body.urdf (robot description, URDF)
Before this commit: robot robot, 5 links, 4 joints
Links:
- link 0: geometry collision box size=0.9433335016429673 0.3220780690035453 0.7671326849483199; visual box size=0.9433335016429673 0.3220780690035453 0.7671326849483199
- link 1: geometry collision box size=1.0896300437428543 0.1860801656466486 0.21184908731298513; visual box size=1.0896300437428543 0.1860801656466486 0.21184908731298513
- link 2: geometry collision box size=1.5539295539971447 0.3218203948088646 0.24444833535798854; visual box size=1.5539295539971447 0.3218203948088646 0.24444833535798854
- link 3: geometry collision box size=0.2390596987112228 0.34153372478832866 0.9266346994815714; visual box size=0.2390596987112228 0.34153372478832866 0.9266346994815714
- link 4: geometry collision box size=0.2760642570256313 1.6026513683114394 0.32296871170588765; visual box size=0.2760642570256313 1.6026513683114394 0.32296871170588765
Joints:
- joint 0_1: axis 1 1 0 -> 0 1 1; origin xyz=0.04001758024304358 0.09857170190427922 0.9849061299035676 rpy=0 0 0 -> xyz=-0.4716667508214836 0.14023979311892593 0.6592000210574291 rpy=0 0 0
- joint 0_2: origin xyz=-0.5605155467243221 -0.1903089767000891 0.6806745243426983 rpy=0 0 0 -> xyz=0.4716667508214836 0.07609134460683536 0.6547221822741912 rpy=0 0 0
- joint 0_3: axis 0 1 1 -> 1 1 0; origin xyz=0.5605155467243221 -0.15534274269175377 0.9060233358558663 rpy=0 0 0 -> xyz=-0.07067575986076335 -0.015378194096255848 0.7671326849483199 rpy=0 0 0
- joint 0_4: origin xyz=-0.39665305309138976 0.2727208375953711 0.17725037835031493 rpy=0 0 0 -> xyz=-0.40979389214158723 -0.16103903450177265 0.6544508423798777 rpy=0 0 0

Commit message: HW8 PHC update

File: body.urdf (robot description, URDF)
Before this commit: robot robot, 5 links, 4 joints
Links:
- added link 5, mass 1; collision box size=1.1505731804979291 0.020079375727397375 0.41316906389359087; visual box size=1.1505731804979291 0.020079375727397375 0.41316906389359087
- added link 6, mass 1; collision box size=0.20423898244386496 1.080398981181843 0.3386928277823188; visual box size=0.20423898244386496 1.080398981181843 0.3386928277823188
- link 0: geometry collision box size=0.6147621059991187 0.36146532803865805 0.5176006051368431; visual box size=0.6147621059991187 0.36146532803865805 0.5176006051368431
- link 1: geometry collision box size=0.43035618573599677 1.0565477029754389 0.21422481829102613; visual box size=0.43035618573599677 1.0565477029754389 0.21422481829102613
- link 2: geometry collision box size=1.0517182317760398 0.26089153259990117 0.17744463114828146; visual box size=1.0517182317760398 0.26089153259990117 0.17744463114828146
- link 3: geometry collision box size=0.4703031966332433 1.4423629211084104 0.3085995344307162; visual box size=0.4703031966332433 1.4423629211084104 0.3085995344307162
- link 4: geometry collision box size=0.3341449737303152 1.4118983458596415 0.08236823055331488; visual box size=0.3341449737303152 1.4118983458596415 0.08236823055331488
Joints:
- added joint 0_5: type revolute, parent 0, child 5, origin xyz=0.30738105299955937 -0.158533331609712 0.24830069464724527 rpy=0 0 0, axis 0 1 1, limit lower=-3.14159 upper=3.14159 effort=0.0 velocity=0.0
- added joint 0_6: type revolute, parent 0, child 6, origin xyz=0.0051322915335622055 -0.18073266401932903 0.30960425502427313 rpy=0 0 0, axis 1 0 1, limit lower=-3.14159 upper=3.14159 effort=0.0 velocity=0.0
- joint 0_1: axis 0 1 1 -> 1 0 1; origin xyz=-0.4716667508214836 0.14023979311892593 0.6592000210574291 rpy=0 0 0 -> xyz=-0.19906948851281378 -0.18073266401932903 0.00479640756710982 rpy=0 0 0
- joint 0_2: origin xyz=0.4716667508214836 0.07609134460683536 0.6547221822741912 rpy=0 0 0 -> xyz=0.30738105299955937 -0.020034747542655107 0.12331103147597434 rpy=0 0 0
- joint 0_3: axis 1 1 0 -> 1 0 1; origin xyz=-0.07067575986076335 -0.015378194096255848 0.7671326849483199 rpy=0 0 0 -> xyz=0.16598774983211273 -0.18073266401932903 0.1333756150976659 rpy=0 0 0
- joint 0_4: origin xyz=-0.40979389214158723 -0.16103903450177265 0.6544508423798777 rpy=0 0 0 -> xyz=0.21454148019838953 -0.18073266401932903 0.09008625755969342 rpy=0 0 0
